Commit message: bot lidar positioning update

File: urdf/simple_bot.urdf.xacro (robot description, xacro)
@@ -69,5 +69,5 @@
   </link>
   <joint name="lidar_joint" type="fixed">
-    <origin xyz="0 0 0.2" rpy="0 0 3.1416"/>
+    <origin xyz="-0.25 0 -0.1" rpy="0 0 3.1416"/>
     <parent link="base_link"/>
     <child link="lidar_link"/>

Commit message: fix lidar clipping

File: urdf/simple_bot.urdf.xacro (robot description, xacro)
@@ -69,5 +69,5 @@
   </link>
   <joint name="lidar_joint" type="fixed">
-    <origin xyz="-0.25 0 -0.1" rpy="0 0 3.1416"/>
+    <origin xyz="-0.26 0 -0.1" rpy="0 0 3.1416"/>
     <parent link="base_link"/>
     <child link="lidar_link"/>

Commit message: remove visualisation of the lidar sensor

File: urdf/simple_bot.urdf.xacro (robot description, xacro)
@@ -62,9 +62,4 @@
   </joint>
   <link name="lidar_link">
-    <visual>
-      <geometry>
-        <cylinder length="0.1" radius="0.1"/>
-      </geometry>
-    </visual>
   </link>
   <joint name="lidar_joint" type="fixed">

Commit message: kind of working

File: urdf/simple_bot.urdf.xacro (robot description, xacro)
@@ -76,5 +76,5 @@
         <scan>
           <horizontal>
-            <samples>1000</samples>
+            <samples>50</samples>
             <resolution>1</resolution>
             <min_angle>-1.570796</min_angle>
@@ -141,6 +141,6 @@
         <horizontal_fov>1.3962634</horizontal_fov>
         <image>
-          <width>640</width>
-          <height>480</height>
+          <width>20</width>
+          <height>20</height>
           <format>R8G8B8</format>
         </image>
@@ -160,3 +160,28 @@
     </sensor>
   </gazebo>
+  <gazebo>
+    <plugin name="gazebo_ros_control" filename="libgazebo_ros_control.so">
+      <robotNamespace>/</robotNamespace>
+    </plugin>
+  </gazebo>
+  <transmission name="left_wheel_trans">
+    <type>transmission_interface/SimpleTransmission</type>
+    <joint name="l_whl_joint">
+      <hardwareInterface>hardware_interface/EffortJointInterface</hardwareInterface>
+    </joint>
+    <actuator name="l_whl_motor">
+      <hardwareInterface>hardware_interface/EffortJointInterface</hardwareInterface>
+      <mechanicalReduction>1</mechanicalReduction>
+    </actuator>
+  </transmission>
+  <transmission name="right_wheel_trans">
+    <type>transmission_interface/SimpleTransmission</type>
+    <joint name="r_whl_joint">
+      <hardwareInterface>hardware_interface/EffortJointInterface</hardwareInterface>
+    </joint>
+    <actuator name="r_whl_motor">
+      <hardwareInterface>hardware_interface/EffortJointInterface</hardwareInterface>
+      <mechanicalReduction>1</mechanicalReduction>
+    </actuator>
+  </transmission>
 </robot>

Commit message: Modify training parameters

File: urdf/simple_bot.urdf.xacro (robot description, xacro)
@@ -20,5 +20,5 @@
     <parent link="base_link"/>
     <child link="l_whl"/>
-    <origin xyz="0 -0.15 0" rpy="1.5708 0 0"/>
+    <origin xyz="0 -0.151 0" rpy="1.5708 0 0"/>
     <axis xyz="0 0 1"/>
   </joint>
@@ -26,10 +26,10 @@
     <visual>
       <geometry>
-        <cylinder radius="0.15" length="0.05"/>
+        <cylinder radius="0.151" length="0.05"/>
       </geometry>
     </visual>
     <collision>
       <geometry>
-        <cylinder radius="0.15" length="0.05"/>
+        <cylinder radius="0.151" length="0.05"/>
       </geometry>
     </collision>
@@ -42,10 +42,10 @@
     <visual>
       <geometry>
-        <cylinder radius="0.15" length="0.05"/>
+        <cylinder radius="0.151" length="0.05"/>
       </geometry>
     </visual>
     <collision>
       <geometry>
-        <cylinder radius="0.15" length="0.05"/>
+        <cylinder radius="0.151" length="0.05"/>
       </geometry>
     </collision>
@@ -58,5 +58,5 @@
     <parent link="base_link"/>
     <child link="r_whl"/>
-    <origin xyz="0 0.15 0" rpy="1.5708 0 0"/>
+    <origin xyz="0 0.151 0" rpy="1.5708 0 0"/>
     <axis xyz="0 0 1"/>
   </joint>
@@ -107,5 +107,5 @@
       <wheelSeparation>0.3</wheelSeparation>
       <wheelDiameter>0.3</wheelDiameter>
-      <torque>10.0</torque>
+      <torque>20.0</torque>
       <commandTopic>cmd_vel</commandTopic>
       <odometryFrame>odom</odometryFrame>
