Commit message: make box pink

File: urdf/pink_box.urdf.xacro (robot description, xacro)
@@ -1,7 +1,4 @@
 <?xml version="1.0"?>
 <robot name="pink_box" xmlns:xacro="http://www.ros.org/wiki/xacro">
-  <material name="pink">
-    <color rgba="1 0.4 0.7 1"/>
-  </material>
   <link name="box_link">
     <visual>
@@ -9,5 +6,4 @@
         <box size="0.3 0.3 0.3"/>
       </geometry>
-      <material name="pink"/>
     </visual>
     <collision>
@@ -24,3 +20,12 @@
     </inertial>
   </link>
+  <gazebo reference="box_link">
+    <visual>
+      <material>
+        <ambient>1 0.4 0.6 1</ambient>
+        <diffuse>1 0 0.6 1</diffuse>
+        <specular>1 0.5 0.7 1</specular>
+      </material>
+    </visual>
+</gazebo>
 </robot>

Commit message: reduce state space

File: urdf/pink_box.urdf.xacro (robot description, xacro)
@@ -4,10 +4,10 @@
     <visual>
       <geometry>
-        <box size="0.3 0.3 0.3"/>
+        <box size="0.7 0.7 0.7"/>
       </geometry>
     </visual>
     <collision>
       <geometry>
-        <box size="0.3 0.3 0.3"/>
+        <box size="0.7 0.7 0.7"/>
       </geometry>
     </collision>
